Commit message: gmapping test_code complete

File: tracer_ros/tracer_description/urdf/tracer_mini.urdf (robot description, URDF)
Before this commit: robot tracer_mini, 16 links, 15 joints
Links:
- link first_floor: geometry collision mesh filename=package://tracer_description/meshes/base/first.stl; visual mesh filename=package://tracer_description/meshes/base/first.stl
- link second_floor: geometry collision mesh filename=package://tracer_description/meshes/base/second.stl; visual mesh filename=package://tracer_description/meshes/base/second.stl
